Commit message: Updates

File: double_pendulum.urdf (robot description, URDF)
Before this commit: robot pendulum, 6 links, 5 joints
Joints:
- joint joint_eef1: origin xyz=0 0 1.5 rpy=0 0 0 -> xyz=0 0 0.8 rpy=0 0 0
- joint joint_eef2: origin xyz=0 0 0.4 rpy=0 0 0 -> xyz=0 0 0.7 rpy=0 0 0

Commit message: upd

File: double_pendulum.urdf (robot description, URDF)
Before this commit: robot pendulum, 6 links, 5 joints
Joints:
- joint joint_1: axis 0 1 0 -> 0 -1 0; origin xyz=0.0 0 0 rpy=0 3.14159265358979323846 0 -> xyz=0.0 0 0 rpy=0 1.5707963267948966 0
- joint joint_2: axis 0 1 0 -> 0 -1 0; origin xyz=0.0 0 0 rpy=0 3.14159265358979323846 0 -> xyz=0.0 0 0 rpy=0 0 0
